File: PIC795MotorBoard.sch (EAGLE design)
At the start: 54 parts, among them J10 MOLEX-2P-156, J11 MOLEX_3P, J12 MOLEX_3P, J13 MOLEX_3P, J14 MOLEX_3P, J21 MOLEX_4PMOLEX_4P, J22 MOLEX_4PMOLEX_4P, J23 MOLEX_4PMOLEX_4P, J24 MOLEX_4PMOLEX_4P, J5 MOLEX_MINI_RA_3P, J6 MOLEX_MINI_RA_3P, J7 MOLEX_MINI_RA_3P, J8 MOLEX_MINI_RA_3P, U1 IFX9201SG, U2 IFX9201SG, U3 IFX9201SG, U4 IFX9201SG

Commit message: Rev 2 board sent to PCB fab 8-11-19
Parts:
- removed C13, C14: 0.1 uF, JimLib:CAP-1206
- removed H2, H4, H5: MOUNT-HOLE3.6, holes:MOUNT-HOLE3.6
- added C10, C9: 0.1 uF, JimLib:CAP-0.300
- added CS, ENABLE, MISO, MOSI, PWM1, PWM2, PWM3, PWM4, SCK: TPTESTPAD-SMALL, JimLib:TPTESTPAD-SMALL
- added R2: 0 Ohm, JimLib:RESISTORR0402
- added U$1, U$2, U$3: FIDUCIAL, adafruit:FIDUCIAL
- C11, C12: device JimLib:CAP-1206 -> JimLib:CAP-0.300
- C15, C16, C17, C18, C19, C20, C21, C22: value 0.022 uF 200V -> 0.022 uF; device JimLib:C0805 -> JimLib:C5/2.5
- D2: value 38.9V -> TRANSZORB
- J5, J6, J7, J8: value MOLEX_MINI_RA_3P -> MOLEX_3PMOLEX-156-3P; device JimLib:MOLEX_MINI_RA_3P -> JimLib:MOLEX_3PMOLEX-156-3P
- R1: value 330 ohms -> 220 ohms; device JimLib:RESISTORR1206 -> JimLib:RESISTOR0204/5
Connections:
- net !SPI_CS: now also CS.TP
- net DISABLE: now also ENABLE.TP
- net ENC1: now also J21.2; no longer J21.3
- net ENC2: now also J22.2; no longer J22.3
- net ENC3: now also J23.2; no longer J23.3
- net ENC4: now also J24.2; no longer J24.3
- net GND: now also C10.1, C11.1, C12.1, C15.1, C16.2, C17.1, C18.2, C19.1, C20.2, C21.1, C22.2, C9.1, J21.3, J22.3, J23.3, J24.3, R2.1, R2.2; no longer C11.2, C12.2, C13.2, C14.2, C15.2, C16.1, C17.2, C18.1, C19.2, C20.1, C21.2, C22.1, J21.2, J22.2, J23.2, J24.2
- net N$10: now also C17.2, J6.3; no longer C18.2, J6.1
- net N$11: now also C20.1, J7.1; no longer C19.1, J7.3
- net N$12: now also C19.2, J7.3; no longer C20.2, J7.1
- net N$13: now also C22.1, J8.1; no longer C21.1, J8.3
- net N$14: now also C21.2, J8.3; no longer C22.2, J8.1
- net N$7: now also C16.1, J5.1; no longer C15.1, J5.3
- net N$8: now also C15.2, J5.3; no longer C16.2, J5.1
- net N$9: now also C18.1, J6.1; no longer C17.1, J6.3
- net OC2: now also PWM1.TP
- net OC3: now also PWM2.TP
- net OC4: now also PWM3.TP
- net OC5: now also PWM4.TP
- net SPI_MISO: now also MISO.TP
- net SPI_MOSI: now also MOSI.TP
- net SPI_SCK: now also SCK.TP
- net VCC: now also C10.2, C11.2, C12.2, C9.2; no longer C11.1, C12.1, C13.1, C14.1
Other:
- note removed: "TODO: ELIMINATE +5V REGULATOR, CONNECT J21-J24 to +3.3V"
- moved on the sheet: C15, C16, C17, C18, C19, C20, C21, C22
